File: PCB/controller_Proto/contProto/contProto.kicad_pcb (KiCad board)
At the start: 4 copper layers, 2.3 x 5.3 mm, 84 parts, among them J1 Conn_01x05, J10 JST_1mm_3, J11 JST_1mm_3, J12 JST_1mm_3, J13 Conn_01x02_Socket, J14 Conn_01x02_Socket, J15 Conn_01x04, J16 Conn_01x04, J17 Conn_01x10_Pin, J18 JST_1mm_3, J19 Conn_01x08_Socket, J2 Conn_01x04, J20 JST_1mm_3, J21 JST_1mm_3, J22 JST_1mm_3, J23 JST_1mm_3, J24 Conn_01x03_Socket, J25 Conn_01x03_Socket, J26 Conn_01x03_Socket, J27 Conn_01x03_Socket, J28 Conn_01x12_Socket, J29 Conn_01x12_Socket, J3 Conn_01x10_Pin, J30 Conn_01x12_Socket, J31 Conn_01x12_Socket, J32 Conn_01x02_Socket, J33 Conn_01x02_Socket, J34 Conn_01x02_Socket, J35 Conn_01x02_Socket, J4 JST_1mm_3, J5 Conn_01x05, J6 JST_1mm_3, J7 Conn_01x05, J8 Conn_01x05, J9 Conn_01x04, SW1 SMD_12x12mm_h8.5mm, SW10 SMD_12x12mm_h8.5mm, SW11 SMD_12x12mm_h8.5mm, SW12 SMD_12x12mm_h8.5mm, SW13 SMD_12x12mm_h8.5mm, SW14 SMD_12x12mm_h8.5mm, SW15 SMD_12x12mm_h8.5mm, SW16 SMD_12x12mm_h8.5mm, SW17 SMD_12x12mm_h8.5mm, SW18 SMD_12x12mm_h8.5mm, SW19 SMD_12x12mm_h8.5mm, SW2 SMD_12x12mm_h8.5mm, SW20 SMD_12x12mm_h8.5mm, SW3 SMD_12x12mm_h8.5mm, SW4 SMD_12x12mm_h8.5mm, SW5 SMD_12x12mm_h8.5mm, SW6 SMD_12x12mm_h8.5mm, SW7 SMD_12x12mm_h8.5mm, SW8 SMD_12x12mm_h8.5mm, SW9 SMD_12x12mm_h8.5mm, U1 ProMicroC, U2 ProMicroC, U3 DRV5033FAxLPG, U4 DRV5033FAxLPG

Commit message: no more errors and trackball ports
Parts:
- removed J13, J14: Conn_01x02_Socket, Connector_PinSocket_1.00mm:PinSocket_1x02_P1.00mm_Vertical
- removed REF**: MouseBite-Slot_2.0x2.0mm_outset_D0.5mm_P0.85mm_3h, Panelization:MouseBite-Slot_2.0x2.0mm_outset_D0.5mm_P0.85mm_3h
- added J36: Conn_01x05, Connector_JST:JST_GH_BM05B-GHS-TBT_1x05-1MP_P1.25mm_Vertical, F.Cu at (51.5, 76.4)
- added J37: Conn_01x05, Connector_JST:JST_GH_BM05B-GHS-TBT_1x05-1MP_P1.25mm_Vertical, F.Cu at (74.6, 21.4)
- moved U4 129.9 mm to (134.6, 28.5), turned to 180 degrees
- moved J25 114.6 mm to (136.0, 39.5), turned to -90 degrees
- moved SW11 106.7 mm to (251.2, 31.7), turned to 0 degrees
- moved SW8 104.4 mm to (239.2, 43.1), turned to -90 degrees
- moved U3 97.7 mm to (119.0, 29.0), turned to 0 degrees
- moved J26 85.3 mm to (118.0, 40.0), turned to 90 degrees
- moved SW10 82.6 mm to (239.2, 18.9), turned to 90 degrees
- moved J1 81.9 mm to (243.7, 64.9)
- moved SW1 81.9 mm to (229.8, 91.4)
- moved SW2 81.9 mm to (241.8, 79.4)
- moved SW3 81.9 mm to (217.7, 80.1)
- moved SW4 81.9 mm to (229.8, 67.4)
- moved SW9 80.7 mm to (227.0, 31.6), turned to 180 degrees
- moved J7 61.5 mm to (220.9, 18.5), turned to 90 degrees
- moved J23 58.5 mm to (159.0, 84.7)
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Connections:
- J28 pad 1: unconnected-(J28-Pin_1-Pad1) -> /tx1
- J28 pad 2: unconnected-(J28-Pin_2-Pad2) -> /Rx1
- J30 pad 1: unconnected-(J30-Pin_1-Pad1) -> /tx2
- J30 pad 2: unconnected-(J30-Pin_2-Pad2) -> /Rx2
- U1 pad 1: unconnected-(U1-TX-Pad1) -> /tx1
- U1 pad 2: unconnected-(U1-RX-Pad2) -> /Rx1
- U2 pad 1: unconnected-(U2-TX-Pad1) -> /tx2
- U2 pad 2: unconnected-(U2-RX-Pad2) -> /Rx2
Routing:
- net SDA: track 72.9 -> 107.9 mm, vias 0 -> 2
- net /Vin: track 34.5 -> 0.58 mm
- net SCL: track 70.5 -> 99.9 mm, vias 0 -> 2
- net /Vin2: track 26.4 -> 0.00 mm
- net VCC2: track 2.20 -> 19.1 mm, vias 7 -> 9
- net /A: track 38.6 -> 39.3 mm
- net VCC: vias 7 -> 8
- net GND: vias 19 -> 21
- net /Btn_A: vias 0 -> 1
Other:
- board size 2.3 x 5.3 mm -> 239.4 x 107.2 mm

Commit message: I almost forgot the mounting holes
Parts:
- added REF**: MountingHole_2.1mm, MountingHole:MountingHole_2.1mm, F.Cu at (174.0, 92.5)
- added REF**: MountingHole_2.5mm_Pad_TopOnly, MountingHole:MountingHole_2.5mm_Pad_TopOnly, F.Cu at (24.5, 20.5)
- added REF**: MountingHole_2.1mm, MountingHole:MountingHole_2.1mm, F.Cu at (159.0, 92.5)
- added REF**: MountingHole_2.1mm, MountingHole:MountingHole_2.1mm, F.Cu at (144.0, 70.5)
- added REF**: MountingHole_2.5mm_Pad_TopOnly, MountingHole:MountingHole_2.5mm_Pad_TopOnly, F.Cu at (108.0, 20.5)
- added REF**: MountingHole_2.1mm, MountingHole:MountingHole_2.1mm, F.Cu at (120.0, 45.0)
- added REF**: MountingHole_2.5mm_Pad_TopOnly, MountingHole:MountingHole_2.5mm_Pad_TopOnly, F.Cu at (253.5, 14.5)
- added REF**: MountingHole_2.5mm_Pad_TopOnly, MountingHole:MountingHole_2.5mm_Pad_TopOnly, F.Cu at (221.5, 44.5)
- added REF**: MountingHole_2.5mm_Pad_TopOnly, MountingHole:MountingHole_2.5mm_Pad_TopOnly, F.Cu at (53.0, 86.0)
- added REF**: MountingHole_2.1mm, MountingHole:MountingHole_2.1mm, F.Cu at (128.5, 70.5)
- added REF**: MountingHole_2.1mm, MountingHole:MountingHole_2.1mm, F.Cu at (81.5, 120.0)
- added REF**: MountingHole_2.1mm, MountingHole:MountingHole_2.1mm, F.Cu at (133.5, 45.0)
- added REF**: MountingHole_2.5mm_Pad_TopOnly, MountingHole:MountingHole_2.5mm_Pad_TopOnly, F.Cu at (244.0, 94.0)
- added REF**: MountingHole_2.1mm, MountingHole:MountingHole_2.1mm, F.Cu at (40.0, 97.0)
- added REF**: MountingHole_2.1mm, MountingHole:MountingHole_2.1mm, F.Cu at (65.0, 108.0)
- added REF**: MountingHole_2.5mm_Pad_TopOnly, MountingHole:MountingHole_2.5mm_Pad_TopOnly, F.Cu at (214.0, 94.0)
- added REF**: MountingHole_2.5mm_Pad_TopOnly, MountingHole:MountingHole_2.5mm_Pad_TopOnly, F.Cu at (253.5, 44.5)
- added REF**: MountingHole_2.1mm, MountingHole:MountingHole_2.1mm, F.Cu at (81.0, 101.3)
- added REF**: MountingHole_2.1mm, MountingHole:MountingHole_2.1mm, F.Cu at (26.0, 109.0)
- added REF**: MountingHole_2.5mm_Pad_TopOnly, MountingHole:MountingHole_2.5mm_Pad_TopOnly, F.Cu at (214.0, 61.0)
- added REF**: MountingHole_2.1mm, MountingHole:MountingHole_2.1mm, F.Cu at (48.0, 97.0)
- moved J15 24.7 mm to (88.2, 100.1)
- moved J27 24.7 mm to (112.1, 103.0)
- moved SW16 24.7 mm to (100.1, 100.5)
- moved J16 21.9 mm to (89.0, 119.6)
- moved J24 21.9 mm to (112.6, 122.0)
- moved SW15 21.9 mm to (101.1, 119.9)
- moved J36 12.0 mm to (39.5, 77.5)
Routing:
- net SCL: track 99.9 -> 112.7 mm
- net SDA: track 107.9 -> 115.1 mm
- net VCC2: track 19.1 -> 25.0 mm
Other:
- board size 239.4 x 107.2 mm -> 239.4 x 115.5 mm

Commit message: move res big v
Parts:
- removed J35: Conn_01x02_Socket, Connector_PinSocket_2.54mm:PinSocket_1x02_P2.54mm_Vertical
- removed R11, R12: 1k, PCM_SparkFun-Resistor:R_0402_1005Metric
- added J13: Conn_01x02_Socket, Connector_PinSocket_2.54mm:PinSocket_1x02_P2.54mm_Vertical, F.Cu at (108.0, 52.5)
- added J14: Conn_01x02_Socket, Connector_PinSocket_2.54mm:PinSocket_1x02_P2.54mm_Vertical, F.Cu at (26.5, 42.5)
- added J38: Conn_01x06, PCM_SparkFun-Connector:JST_1x06_P1.0mm_Horizontal_SMD, B.Cu at (243.0, 62.5)
- J1: value Conn_01x05 -> JST_1mm_4; footprint Connector_JST:JST_GH_BM05B-GHS-TBT_1x05-1MP_P1.25mm_Vertical -> PCM_SparkFun-Connector:JST_1x04_P1.0mm_Horizontal_SMD
- J12, J23: value JST_1mm_3 -> Conn_01x03_Socket; footprint Connector_JST:JST_GH_BM03B-GHS-TBT_1x03-1MP_P1.25mm_Vertical -> Connector_PinSocket_2.54mm:PinSocket_1x03_P2.54mm_Vertical; moved to F.Cu
- J22, J4: value JST_1mm_3 -> JST_1mm_4; footprint Connector_JST:JST_GH_BM03B-GHS-TBT_1x03-1MP_P1.25mm_Vertical -> PCM_SparkFun-Connector:JST_1x04_P1.0mm_Horizontal_SMD
- J32, J33: value Conn_01x02_Socket -> Conn_01x03_Socket; footprint Connector_PinSocket_2.54mm:PinSocket_1x02_P2.54mm_Vertical -> Connector_PinSocket_2.54mm:PinSocket_1x03_P2.54mm_Vertical
- J34: value Conn_01x02_Socket -> JST_1mm_4; footprint Connector_PinSocket_2.54mm:PinSocket_1x02_P2.54mm_Vertical -> PCM_SparkFun-Connector:JST_1x04_P1.0mm_Horizontal_SMD; moved to B.Cu
- J7: value Conn_01x05 -> Conn_01x06; footprint Connector_JST:JST_GH_BM05B-GHS-TBT_1x05-1MP_P1.25mm_Vertical -> PCM_SparkFun-Connector:JST_1x06_P1.0mm_Horizontal_SMD
- R13, R14, R16, R18, R19, R21, R5, R6, R7, R8: moved to F.Cu
- moved R6 189.7 mm to (236.2, 26.8), turned to -90 degrees
- moved R16 188.5 mm to (242.5, 32.2)
- moved R7 179.8 mm to (231.5, 32.2), turned to 0 degrees
- moved R21 178.8 mm to (236.0, 37.5), turned to 90 degrees
- moved R8 177.7 mm to (235.0, 79.5), turned to 180 degrees
- moved R5 173.5 mm to (225.0, 80.0), turned to 0 degrees
- moved R18 171.9 mm to (229.5, 84.5)
- moved R14 150.4 mm to (229.5, 74.0)
- moved J12 135.9 mm to (155.7, 63.0), turned to 90 degrees
- moved R17 111.9 mm to (163.7, 76.0), turned to 0 degrees
- moved R4 98.6 mm to (178.2, 77.5)
- moved R2 86.7 mm to (20.8, 104.5)
- moved J1 86.3 mm to (159.2, 82.4), turned to 180 degrees
- moved R15 75.4 mm to (147.0, 80.0), turned to 0 degrees
- moved R1 70.5 mm to (132.2, 79.8), turned to 180 degrees
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Connections:
- J1 pad 1: /FB_VCC -> /PPGND
- J1 pad 2: /Btn_Y -> /PPVCC1
- J1 pad 3: /Btn_X -> /PP1
- J1 pad 4: /Btn_B -> /PP2
- J12 pad 1: /SL_VCC -> /PP2
- J12 pad 2: /Btn_SP3 -> /PPVCC1
- J12 pad 3: /Btn_- -> /PPGND
- J22 pad 1: /PPVCC2 -> /PPGND2
- J22 pad 2: /PP3 -> /PPVCC2
- J22 pad 3: /PP4 -> /PP3
- J23 pad 1: /PPVCC1 -> /PP4
- J23 pad 2: /PP1 -> /PPVCC2
- J23 pad 3: /PP2 -> /PPGND2
- J32 pad 1: /PP4 -> /PP42
- J32 pad 2: /PPVCC2 -> /PPVCC22
- J33 pad 1: /PP2 -> /PP22
- J33 pad 2: /PPVCC1 -> /PPVCC12
- J34 pad 1: /PP42 -> /SR_GND
- J34 pad 2: /PPVCC22 -> /SR_VCC
- J4 pad 1: /SR_VCC -> /SL_GND
- J4 pad 2: /Btn_+ -> /SL_VCC
- J4 pad 3: /Btn_SP2 -> /Btn_SP3
- J7 pad 1: /D_VCC -> /D_GND
- J7 pad 2: /Btn_U -> /D_VCC
- J7 pad 3: /Btn_L -> /Btn_U
- J7 pad 4: /Btn_R -> /Btn_L
- J7 pad 5: /Btn_D -> /Btn_R
- R1 pad 1: /X -> /PP42
- R1 pad 2: GND -> /PPGND22
- R10 pad 1: /Pad2 -> /R1P
- R10 pad 2: GND -> GND_RSP
- R14 pad 1: /B -> /Btn_A
- R14 pad 2: GND -> /FB_GND
- R15 pad 1: /Pad1 -> /PP22
- R15 pad 2: GND -> /PPGND12
- R16 pad 1: /R -> /Btn_R
- R16 pad 2: GND -> /D_GND
- R17 pad 1: /Pad3 -> /PP1
- R17 pad 2: GND -> /PPGND
- R18 pad 1: /Btn2 -> /Btn_Y
- R18 pad 2: GND -> /FB_GND
- R2 pad 1: /Y -> /Btn_-
- R2 pad 2: GND -> /SL_GND
- R20 pad 1: /SP2 -> /Btn_+
- R20 pad 2: GND -> /SR_GND
- R21 pad 1: /D -> /Btn_D
- R21 pad 2: GND -> /D_GND
- R22 pad 1: /plus -> /Btn_SP2
- R22 pad 2: GND -> /SR_GND
- R3 pad 1: /L1 -> /L1P
- R3 pad 2: GND -> GND_LSP
- R4 pad 1: /A -> /PP3
- R4 pad 2: GND -> /PPGND2
- R5 pad 1: /SP3 -> /Btn_B
- R5 pad 2: GND -> /FB_GND
- R6 pad 1: /U -> /Btn_U
- R6 pad 2: GND -> /D_GND
- R7 pad 1: /L -> /Btn_L
- R7 pad 2: GND -> /D_GND
- R8 pad 1: /minus -> /Btn_X
- R8 pad 2: GND -> /FB_GND
- R9 pad 1: /R1 -> /Btn_SP3
- R9 pad 2: GND -> /SL_GND
Routing:
- net /SR_VCC: track 0.00 -> 42.7 mm, vias 3 -> 2
- net /Btn_Y: track 26.3 -> 58.3 mm
- net /SL_GND: track 0.00 -> 26.0 mm
- net VCC_LSP: track 0.00 -> 25.9 mm, vias 1 -> 2
- net /PPGND: track 0.00 -> 25.2 mm
- net VCC_RSP: track 0.00 -> 24.9 mm
- net /SL_VCC: track 0.00 -> 23.8 mm, vias 3 -> 2
- net /PPGND2: track 0.00 -> 21.6 mm
- net /SR_GND: track 0.00 -> 20.5 mm
- net /plus: track 40.6 -> 55.6 mm, vias 2 -> 1
- net GND: track 57.4 -> 43.7 mm, vias 21 -> 9
- net GND_RSP: track 21.9 -> 35.0 mm, vias 1 -> 0
- net /R2: track 50.8 -> 38.5 mm
- net /PP1: track 11.3 -> 22.9 mm
- net /SP2: track 42.2 -> 53.7 mm, vias 2 -> 0
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- added copper zone on In2.Cu, net /D_GND
- added copper zone on In2.Cu, net /FB_GND
- added copper zone on In2.Cu, net GND
- removed copper zone on B.Cu, net /SL_VCC
- removed copper zone on B.Cu, net /SR_VCC
- removed copper zone on F.Cu, net GND
- removed copper zone on B.Cu, net VCC_LSP
- removed copper zone on B.Cu, net VCC_RSP
Other:
- board size 239.4 x 115.5 mm -> 237.9 x 117 mm
