File: PCB/controller_Proto/contProto2/contProto.kicad_pcb (KiCad board)
At the start: 4 copper layers, 64.8 x 107 mm, 82 parts, among them J1 JST_1mm_4, J10 JST_1mm_3, J11 JST_1mm_3, J12 Conn_01x03_Socket, J13 Conn_01x02_Socket, J14 Conn_01x02_Socket, J15 Conn_01x04, J16 Conn_01x04, J17 Conn_01x10_Pin, J18 JST_1mm_3, J19 Conn_01x08_Socket, J2 Conn_01x04, J22 JST_1mm_4, J23 Conn_01x03_Socket, J24 Conn_01x03_Socket, J25 Conn_01x03_Socket, J26 Conn_01x03_Socket, J27 Conn_01x03_Socket, J28 Conn_01x12_Socket, J29 Conn_01x12_Socket, J3 Conn_01x10_Pin, J30 Conn_01x12_Socket, J31 Conn_01x12_Socket, J32 Conn_01x03_Socket, J33 Conn_01x03_Socket, J36 Conn_01x05, J37 Conn_01x05, J4 JST_1mm_3, J5 Conn_01x02_Socket, J6 JST_1mm_3, J7 Conn_01x02_Socket, J9 Conn_01x04, SW1 SMD_12x12mm_h8.5mm, SW10 SMD_12x12mm_h8.5mm, SW11 SMD_12x12mm_h8.5mm, SW12 SMD_12x12mm_h8.5mm, SW13 SMD_12x12mm_h8.5mm, SW14 SMD_12x12mm_h8.5mm, SW15 SMD_12x12mm_h8.5mm, SW16 SMD_12x12mm_h8.5mm, SW17 SMD_12x12mm_h8.5mm, SW18 SMD_12x12mm_h8.5mm, SW19 SMD_12x12mm_h8.5mm, SW2 SMD_12x12mm_h8.5mm, SW20 SMD_12x12mm_h8.5mm, SW3 SMD_12x12mm_h8.5mm, SW4 SMD_12x12mm_h8.5mm, SW5 SMD_12x12mm_h8.5mm, SW6 SMD_12x12mm_h8.5mm, SW7 SMD_12x12mm_h8.5mm, SW8 SMD_12x12mm_h8.5mm, SW9 SMD_12x12mm_h8.5mm, U1 ProMicroC, U2 ProMicroC, U3 DRV5033FAxLPG, U4 DRV5033FAxLPG

Commit message: MAJOR PCB REDESIGN
shit here we go again
Parts:
- added REF**: MountingHole_2.5mm_Pad, MountingHole:MountingHole_2.5mm_Pad, F.Cu at (67.0, 68.5)
- added REF**: MountingHole_2.5mm_Pad, MountingHole:MountingHole_2.5mm_Pad, F.Cu at (47.2, 42.8)
- moved J4 34.4 mm to (44.9, 116.2), turned to 90 degrees
- moved J18 28.5 mm to (45.2, 136.8)
- moved J37 18.5 mm to (80.0, 136.2)
- moved J13 16.6 mm to (50.2, 101.5), turned to 0 degrees
- moved J28 16.5 mm to (57.5, 123.8)
- moved J29 16.5 mm to (76.2, 95.8)
- moved U1 16.5 mm to (66.9, 111.0)
- moved J10 15.4 mm to (56.5, 136.5)
- moved R2 7.12 mm to (33.8, 54.2), turned to 0 degrees
- moved SW7 6.41 mm to (33.2, 46.8), turned to 90 degrees
- moved TP4 5.59 mm to (43.5, 101.0), turned to 90 degrees
- moved R20 5.31 mm to (30.0, 39.2)
- moved SW5 5.30 mm to (33.4, 35.0)
- moved R19 4.88 mm to (84.8, 102.1)
- moved SW18 4.88 mm to (84.8, 94.9)
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Connections:
- J29 pad 5: /Xout -> /Yout
- J29 pad 6: /Yout -> /Xout
- U1 pad 17: /Xout -> /Yout
- U1 pad 18: /Yout -> /Xout
Routing:
- net /Vin: track 35.3 -> 0.00 mm
- net VCC: track 1.81 -> 32.8 mm, vias 12 -> 13
- net /Pad1: track 36.1 -> 62.9 mm, vias 1 -> 0
- net /Xout: track 33.2 -> 12.0 mm
- net /RST1: track 14.0 -> 33.8 mm
- net /Y: track 58.5 -> 77.1 mm
- net /R2: track 77.9 -> 96.2 mm, vias 0 -> 1
- net /B: track 55.7 -> 73.1 mm
- net /A: track 52.1 -> 66.7 mm
- net /plus: track 75.8 -> 89.4 mm
- net /X: track 43.9 -> 57.2 mm
- net /R1: track 66.4 -> 77.8 mm, vias 0 -> 1
- net /Btn: track 49.0 -> 37.8 mm, vias 0 -> 1
- net /Yout: track 23.0 -> 12.4 mm, vias 1 -> 0
- net /SP2: track 66.1 -> 75.9 mm
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Other:
- board size 64.8 x 107 mm -> 66 x 120 mm

Commit message: final resesign and silk screen
Parts:
- removed the REF** at (67.0, 68.5)
- removed the REF** at (85.2, 125.5)
- removed the REF** at (47.2, 42.8)
- removed TP1, TP4: TestPoint_2Pole, TestPoint:TestPoint_Bridge_Pitch2.0mm_Drill0.7mm
- added J8: JST_1mm_4, Connector_JST:JST_GH_BM04B-GHS-TBT_1x04-1MP_P1.25mm_Vertical, B.Cu at (86.8, 123.0)
- added REF**: MountingHole_2.5mm_Pad, MountingHole:MountingHole_2.5mm_Pad, F.Cu at (143.5, 68.2)
- added REF**: MPU, MountingHole:MountingHole_2.5mm_Pad, F.Cu at (103.7, 46.5)
- added REF**: MountingHole_2.5mm_Pad, MountingHole:MountingHole_2.5mm_Pad, F.Cu at (143.5, 42.8)
- added SPL: JST_1mm_4, Connector_JST:JST_GH_BM04B-GHS-TBT_1x04-1MP_P1.25mm_Vertical, B.Cu at (103.0, 36.2)
- J1, J22: footprint PCM_SparkFun-Connector:JST_1x04_P1.0mm_Horizontal_SMD -> Connector_JST:JST_GH_BM04B-GHS-TBT_1x04-1MP_P1.25mm_Vertical; moved to B.Cu
- J15, J16, J30, J31, R17, R4, U2: moved to B.Cu
- L_Joy: renamed from J17; moved to B.Cu
- L_shoulder: renamed from J9; moved to B.Cu
- MPU: renamed from J19; moved to B.Cu
- PAD: renamed from J6; moved to B.Cu
- RST: renamed from SW17; moved to B.Cu
- Rumble: renamed from J11; moved to B.Cu
- TRACK_B: renamed from J36; moved to B.Cu
- Vin: renamed from J14; moved to B.Cu
- moved J22 231.0 mm to (27.5, 121.7), turned to 180 degrees
- moved J32 230.8 mm to (29.7, 92.8), turned to -90 degrees
- moved J33 222.3 mm to (43.1, 92.8), turned to -90 degrees
- moved R4 220.4 mm to (25.0, 117.8)
- moved J1 219.8 mm to (40.8, 121.4), turned to 180 degrees
- moved J23 214.3 mm to (29.8, 109.2), turned to -90 degrees
- moved R1 212.1 mm to (29.9, 96.8), turned to 180 degrees
- moved R17 210.1 mm to (40.7, 117.0)
- moved J27 208.5 mm to (53.0, 105.5), turned to 90 degrees
- moved R15 202.8 mm to (44.2, 96.2), turned to 180 degrees
- moved J12 202.6 mm to (38.0, 109.2), turned to 90 degrees
- moved U4 193.6 mm to (57.0, 84.5)
- moved J25 192.9 mm to (55.5, 92.2), turned to 90 degrees
- moved R3 192.5 mm to (52.5, 110.5)
- moved J15 192.5 mm to (55.6, 123.7)
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- renumbered SW4 to A, SW3 to B, J5 to CAP?, SW10 to DWN, J4 to I2C, J13 to JVin, SW8 to L, SW5 to MINUS, J18 to PAD, SW11 to R, SW18 to RST, J10 to RUMBLE, J3 to R_JOY, J2 to R_SHOULDER, SW7 to SP1, J37 to TRACK_B, SW9 to UP, SW2 to X, SW1 to Y, J7 to cap?
Connections:
- J29 pad 1: /SP2 -> /plus
- J29 pad 2: /plus -> /SP2
- J31 pad 2: unconnected-(J31-Pin_2-Pad2) -> GND2
- R pad 1: unconnected-(SW11-Pad1) -> /R
- R22 pad 1: /minus -> /Btn_-
- R22 pad 2: GND2 -> SL_GND
- R9 pad 1: /SP3 -> /Btn_SP3
- R9 pad 2: GND2 -> SL_GND
- SW12 pad 2: VCC2 -> SL_VCC
- SW14 pad 2: VCC2 -> SL_VCC
- U1 pad 13: /SP2 -> /plus
- U1 pad 14: /plus -> /SP2
Routing:
- net SDA2: track 0.00 -> 68.8 mm
- net /R1: track 77.8 -> 19.3 mm, vias 1 -> 0
- net /plus: track 89.4 -> 33.8 mm
- net SCL2: track 0.00 -> 54.9 mm
- net /R2: track 96.2 -> 42.3 mm
- net /A: track 66.7 -> 19.0 mm
- net /Vin2: track 0.00 -> 46.8 mm, vias 0 -> 1
- net /Y: track 77.1 -> 30.5 mm
- net GND2: track 0.00 -> 45.3 mm, vias 0 -> 7
- net /RST2: track 0.00 -> 44.7 mm, vias 0 -> 1
- net /B: track 73.1 -> 29.2 mm
- net /SP2: track 75.9 -> 36.9 mm
- net /X: track 57.2 -> 18.8 mm
- net /L1: track 0.00 -> 35.3 mm
- net /Btn2: track 0.00 -> 34.5 mm, vias 0 -> 1
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- added copper zone on B.Cu, net GND2
- added copper zone on F.Cu, net VCC
- added copper zone on F.Cu, net VCC2
- removed copper zone on In2.Cu, net VCC
Other:
- board size 66 x 120 mm -> 125.6 x 105 mm
- copper layers 4 -> 2
- board text added: "L"
- board text added: "R"

Commit message: Big resistors
Parts:
- R1, R10, R13, R14, R15, R16, R17, R18, R19, R2, R20, R21, R22, R3, R4, R5, R6, R7, R8, R9: footprint PCM_SparkFun-Resistor:R_0402_1005Metric -> PCM_SparkFun-Resistor:R_0805_2012Metric
- moved U4 13.9 mm to (56.3, 98.4), turned to 180 degrees
- moved U3 13.0 mm to (71.3, 97.5), turned to 180 degrees
- moved R16 9.64 mm to (144.5, 56.8)
- moved R21 8.97 mm to (141.2, 58.8)
- moved R7 6.96 mm to (131.0, 49.8)
- moved J11 6.92 mm to (146.7, 62.1)
- moved J14 6.92 mm to (130.3, 67.8)
- moved J17 6.92 mm to (109.1, 32.2)
- moved J19 6.92 mm to (104.2, 47.1)
- moved J20 6.92 mm to (108.2, 40.8)
- moved J36 6.92 mm to (110.5, 70.5)
- moved J6 6.92 mm to (121.8, 70.5)
- moved J7 6.92 mm to (118.8, 38.8)
- moved J9 6.92 mm to (121.4, 31.7)
- moved REF** 6.92 mm to (109.0, 51.0)
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- gave numbers to parts that had none: 2
- renumbered RUMBLE to J10, Rumble to J11, JVin to J13, Vin to J14, L_Joy to J17, PAD to J18, MPU to J19, R_SHOULDER to J2, SPL to J20, R_JOY to J3, TRACK_B to J36, TRACK_B to J37, I2C to J4, PAD to J6, L_shoulder to J9, Y to SW1, DWN to SW10, R to SW11, RST to SW17, RST to SW18, X to SW2, B to SW3, A to SW4, MINUS to SW5, SP1 to SW7, L to SW8, UP to SW9
Routing:
- net VCC2: track 22.2 -> 49.5 mm
- net GND: track 20.6 -> 28.8 mm
- net /R: track 15.2 -> 17.4 mm
- net /D: track 9.13 -> 11.2 mm
- net /X: track 18.8 -> 20.3 mm
- net GND2: track 45.3 -> 43.9 mm, vias 7 -> 6
- net /PPGND2: track 16.3 -> 17.7 mm
- net /A: track 19.0 -> 20.3 mm
- net SL_VCC: track 23.4 -> 24.6 mm
- net /PP1: track 10.9 -> 11.9 mm
- net /Vin2: track 46.8 -> 47.8 mm
- net VCC: vias 11 -> 6
- net /Pad4: vias 1 -> 0
Other:
- board size 125.6 x 105 mm -> 130.9 x 105.1 mm

Commit message: final pcb
Parts:
- removed J1, J20, J22, J8: JST_1mm_4, Connector_JST:JST_GH_BM04B-GHS-TBT_1x04-1MP_P1.25mm_Vertical
- removed J15, J16, J2: Conn_01x04, Connector_JST:JST_GH_BM04B-GHS-TBT_1x04-1MP_P1.25mm_Vertical
- removed J36: Conn_01x05, Connector_JST:JST_GH_BM05B-GHS-TBT_1x05-1MP_P1.25mm_Vertical
- removed J6: JST_1mm_3, Connector_JST:JST_GH_BM03B-GHS-TBT_1x03-1MP_P1.25mm_Vertical
- added JP1: ~, PCM_SparkFun-Jumper:Jumper_3_NO, F.Cu at (99.9, 61.5)
- added JP2: ~, PCM_SparkFun-Jumper:Jumper_3_NO, F.Cu at (45.0, 63.7)
- added L_SHOUL1: Conn_01x04, Connector_FFC-FPC:Amphenol_F32Q-1A7x1-11004_1x04-1MP_P0.5mm_Horizontal, B.Cu at (93.7, 99.8)
- added PAD3: Conn_01x04, Connector_FFC-FPC:Amphenol_F32Q-1A7x1-11004_1x04-1MP_P0.5mm_Horizontal, B.Cu at (35.8, 61.8)
- added PAD4: Conn_01x04, Connector_FFC-FPC:Amphenol_F32Q-1A7x1-11004_1x04-1MP_P0.5mm_Horizontal, B.Cu at (114.2, 73.6)
- added PAD_B1: Conn_01x04, Connector_FFC-FPC:Amphenol_F32Q-1A7x1-11004_1x04-1MP_P0.5mm_Horizontal, B.Cu at (118.3, 98.7)
- added PAD_B2: Conn_01x04, Connector_FFC-FPC:Amphenol_F32Q-1A7x1-11004_1x04-1MP_P0.5mm_Horizontal, B.Cu at (140.9, 98.5)
- added R12: 1k, PCM_SparkFun-Resistor:R_0805_2012Metric, F.Cu at (52.4, 68.0)
- added R23: 1k, PCM_SparkFun-Resistor:R_0805_2012Metric, F.Cu at (56.4, 71.4)
- added R24: 1k, PCM_SparkFun-Resistor:R_0805_2012Metric, F.Cu at (103.7, 70.2)
- added R25: 1k, PCM_SparkFun-Resistor:R_0805_2012Metric, F.Cu at (105.5, 74.8)
- added R26: 1k, PCM_SparkFun-Resistor:R_0805_2012Metric, F.Cu at (56.5, 69.1)
- added R27: 1k, PCM_SparkFun-Resistor:R_0805_2012Metric, F.Cu at (108.2, 74.8)
- added REF**: MouseBite-Slot_2.54x2.54mm_on-edge_D0.5mm_P0.85mm_4h_Trace, Panelization:MouseBite-Slot_2.54x2.54mm_on-edge_D0.5mm_P0.85mm_4h_Trace, F.Cu at (52.5, 92.3)
- added REF**: MouseBite-Slot_2.54x2.54mm_on-edge_D0.5mm_P0.85mm_4h_Trace, Panelization:MouseBite-Slot_2.54x2.54mm_on-edge_D0.5mm_P0.85mm_4h_Trace, F.Cu at (64.5, 92.2)
- added REF**: MouseBite-Slot_2.54x2.54mm_on-edge_D0.5mm_P0.85mm_4h_Trace, Panelization:MouseBite-Slot_2.54x2.54mm_on-edge_D0.5mm_P0.85mm_4h_Trace, F.Cu at (137.2, 90.4)
- added REF**: MouseBite-Slot_2.54x2.54mm_on-edge_D0.5mm_P0.85mm_4h_Trace, Panelization:MouseBite-Slot_2.54x2.54mm_on-edge_D0.5mm_P0.85mm_4h_Trace, F.Cu at (122.4, 78.4)
- added REF**: MouseBite-Slot_2.54x2.54mm_on-edge_D0.5mm_P0.85mm_4h_Trace, Panelization:MouseBite-Slot_2.54x2.54mm_on-edge_D0.5mm_P0.85mm_4h_Trace, F.Cu at (124.4, 99.0)
- added REF**: MouseBite-Slot_2.54x2.54mm_on-edge_D0.5mm_P0.85mm_4h_Trace, Panelization:MouseBite-Slot_2.54x2.54mm_on-edge_D0.5mm_P0.85mm_4h_Trace, F.Cu at (50.0, 106.2)
- added REF**: MouseBite-Slot_2.54x2.54mm_on-edge_D0.5mm_P0.85mm_4h_Trace, Panelization:MouseBite-Slot_2.54x2.54mm_on-edge_D0.5mm_P0.85mm_4h_Trace, F.Cu at (106.8, 104.0)
- added REF**: MouseBite-Slot_2.54x2.54mm_on-edge_D0.5mm_P0.85mm_4h_Trace, Panelization:MouseBite-Slot_2.54x2.54mm_on-edge_D0.5mm_P0.85mm_4h_Trace, F.Cu at (93.0, 34.2)
- added REF**: MouseBite-Slot_2.54x2.54mm_on-edge_D0.5mm_P0.85mm_4h_Trace, Panelization:MouseBite-Slot_2.54x2.54mm_on-edge_D0.5mm_P0.85mm_4h_Trace, F.Cu at (93.0, 53.2)
- added REF**: MouseBite-Slot_2.54x2.54mm_on-edge_D0.5mm_P0.85mm_4h_Trace, Panelization:MouseBite-Slot_2.54x2.54mm_on-edge_D0.5mm_P0.85mm_4h_Trace, F.Cu at (129.0, 104.2)
- added REF**: MouseBite-Slot_2.54x2.54mm_on-edge_D0.5mm_P0.85mm_4h_Trace, Panelization:MouseBite-Slot_2.54x2.54mm_on-edge_D0.5mm_P0.85mm_4h_Trace, F.Cu at (79.5, 85.7)
- added REF**: MouseBite-Slot_2.54x2.54mm_on-edge_D0.5mm_P0.85mm_4h_Trace, Panelization:MouseBite-Slot_2.54x2.54mm_on-edge_D0.5mm_P0.85mm_4h_Trace, F.Cu at (67.8, 78.2)
- added REF**: MouseBite-Slot_2.54x2.54mm_on-edge_D0.5mm_P0.85mm_4h_Trace, Panelization:MouseBite-Slot_2.54x2.54mm_on-edge_D0.5mm_P0.85mm_4h_Trace, F.Cu at (77.2, 105.3)
- added REF**: MouseBite-Slot_2.54x2.54mm_on-edge_D0.5mm_P0.85mm_4h_Trace, Panelization:MouseBite-Slot_2.54x2.54mm_on-edge_D0.5mm_P0.85mm_4h_Trace, F.Cu at (51.5, 78.2)
- added REF**: MouseBite-Slot_2.54x2.54mm_on-edge_D0.5mm_P0.85mm_4h_Trace, Panelization:MouseBite-Slot_2.54x2.54mm_on-edge_D0.5mm_P0.85mm_4h_Trace, F.Cu at (90.8, 105.3)
- added REF**: MouseBite-Slot_2.54x2.54mm_on-edge_D0.5mm_P0.85mm_4h_Trace, Panelization:MouseBite-Slot_2.54x2.54mm_on-edge_D0.5mm_P0.85mm_4h_Trace, F.Cu at (112.6, 85.5)
- added REF**: MouseBite-Slot_2.54x2.54mm_on-edge_D0.5mm_P0.85mm_4h_Trace, Panelization:MouseBite-Slot_2.54x2.54mm_on-edge_D0.5mm_P0.85mm_4h_Trace, F.Cu at (93.0, 73.2)
- added REF**: MouseBite-Slot_2.54x2.54mm_on-edge_D0.5mm_P0.85mm_4h_Trace, Panelization:MouseBite-Slot_2.54x2.54mm_on-edge_D0.5mm_P0.85mm_4h_Trace, F.Cu at (138.3, 78.4)
- added REF**: MouseBite-Slot_2.54x2.54mm_on-edge_D0.5mm_P0.85mm_4h_Trace, Panelization:MouseBite-Slot_2.54x2.54mm_on-edge_D0.5mm_P0.85mm_4h_Trace, F.Cu at (139.4, 106.7)
- added REF**: MouseBite-Slot_2.54x2.54mm_on-edge_D0.5mm_P0.85mm_4h_Trace, Panelization:MouseBite-Slot_2.54x2.54mm_on-edge_D0.5mm_P0.85mm_4h_Trace, F.Cu at (85.8, 91.5)
- added REF**: MouseBite-Slot_2.54x2.54mm_on-edge_D0.5mm_P0.85mm_4h_Trace, Panelization:MouseBite-Slot_2.54x2.54mm_on-edge_D0.5mm_P0.85mm_4h_Trace, F.Cu at (85.2, 78.2)
- added REF**: MouseBite-Slot_2.54x2.54mm_on-edge_D0.5mm_P0.85mm_4h_Trace, Panelization:MouseBite-Slot_2.54x2.54mm_on-edge_D0.5mm_P0.85mm_4h_Trace, F.Cu at (108.4, 91.2)
- added REF**: MouseBite-Slot_2.54x2.54mm_on-edge_D0.5mm_P0.85mm_4h_Trace, Panelization:MouseBite-Slot_2.54x2.54mm_on-edge_D0.5mm_P0.85mm_4h_Trace, F.Cu at (99.1, 113.1)
- added REF**: MouseBite-Slot_2.54x2.54mm_on-edge_D0.5mm_P0.85mm_4h_Trace, Panelization:MouseBite-Slot_2.54x2.54mm_on-edge_D0.5mm_P0.85mm_4h_Trace, F.Cu at (72.5, 99.2)
- added REF**: MouseBite-Slot_2.54x2.54mm_on-edge_D0.5mm_P0.85mm_4h_Trace, Panelization:MouseBite-Slot_2.54x2.54mm_on-edge_D0.5mm_P0.85mm_4h_Trace, F.Cu at (107.3, 78.4)
- added REF**: MouseBite-Slot_2.54x2.54mm_on-edge_D0.5mm_P0.85mm_4h_Trace, Panelization:MouseBite-Slot_2.54x2.54mm_on-edge_D0.5mm_P0.85mm_4h_Trace, F.Cu at (130.9, 85.7)
- added REF**: MouseBite-Slot_2.54x2.54mm_on-edge_D0.5mm_P0.85mm_4h_Trace, Panelization:MouseBite-Slot_2.54x2.54mm_on-edge_D0.5mm_P0.85mm_4h_Trace, F.Cu at (64.2, 106.2)
- added R_SHOUL1: Conn_01x04, Connector_FFC-FPC:Amphenol_F32Q-1A7x1-11004_1x04-1MP_P0.5mm_Horizontal, B.Cu at (48.7, 100.4)
- added R_SHOULD1: Conn_01x04, Connector_FFC-FPC:Amphenol_F32Q-1A7x1-11004_1x04-1MP_P0.5mm_Horizontal, B.Cu at (47.5, 26.0)
- added SP_L1: Conn_01x04, Connector_FFC-FPC:Amphenol_F32Q-1A7x1-11004_1x04-1MP_P0.5mm_Horizontal, B.Cu at (96.5, 42.4)
- added SP_LB1: Conn_01x04, Connector_FFC-FPC:Amphenol_F32Q-1A7x1-11004_1x04-1MP_P0.5mm_Horizontal, B.Cu at (48.5, 86.5)
- added TRACK_B1: Conn_01x05, Connector_PinHeader_2.54mm:PinHeader_1x05_P2.54mm_Vertical, B.Cu at (100.0, 65.0)
- J11: footprint Connector_JST:JST_GH_BM03B-GHS-TBT_1x03-1MP_P1.25mm_Vertical -> Connector_PinHeader_2.54mm:PinHeader_1x03_P2.54mm_Vertical; moved to F.Cu
- J9: footprint Connector_JST:JST_GH_BM04B-GHS-TBT_1x04-1MP_P1.25mm_Vertical -> Connector_FFC-FPC:Amphenol_F32Q-1A7x1-11004_1x04-1MP_P0.5mm_Horizontal
- RUMBLE1: renamed from J10; footprint Connector_JST:JST_GH_BM03B-GHS-TBT_1x03-1MP_P1.25mm_Vertical -> Connector_PinHeader_2.54mm:PinHeader_1x03_P2.54mm_Vertical
- TRACK_B2: renamed from J37; value Conn_01x05 -> TRACK_B; footprint Connector_JST:JST_GH_BM05B-GHS-TBT_1x05-1MP_P1.25mm_Vertical -> Connector_PinHeader_2.54mm:PinHeader_1x05_P2.54mm_Vertical
- moved R4 109.9 mm to (135.4, 98.8), turned to 90 degrees
- moved SW19 105.8 mm to (131.9, 98.6), turned to 90 degrees
- moved J23 97.8 mm to (126.7, 96.2), turned to 0 degrees
- moved SW20 84.5 mm to (110.1, 86.0), turned to -90 degrees
- moved R1 78.2 mm to (106.8, 83.0), turned to -90 degrees
- moved J32 73.8 mm to (102.9, 83.1), turned to 0 degrees
- moved R17 73.7 mm to (112.1, 98.7), turned to 90 degrees
- moved LT1 71.1 mm to (141.2, 84.6), turned to -90 degrees
- moved RT1 70.2 mm to (125.2, 84.9), turned to -90 degrees
- moved PAD1 69.6 mm to (108.6, 98.8), turned to 90 degrees
- moved J12 66.6 mm to (104.1, 101.5), turned to 180 degrees
- moved J26 60.8 mm to (133.2, 83.2), turned to 0 degrees
- moved J25 60.1 mm to (117.5, 83.4), turned to 0 degrees
- moved J18 56.9 mm to (107.7, 62.1), turned to -45 degrees
- moved PAD2 50.2 mm to (89.3, 86.2), turned to -90 degrees
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- renumbered SW4 to A1, SW3 to B1, J5 to CAP1, J7 to CAP2, SW10 to DWN1, J4 to I2C1, J3 to JOY_R1, SW8 to L1, SW16 to LB1, U3 to LT1, SW12 to MINUS1, J19 to MPU1, SW13 to PAD1, SW6 to PAD2, SW5 to PLUS1, SW11 to R11, SW15 to RB1, SW17 to RST1, SW18 to RST2, U4 to RT1, SW7 to SP1, SW14 to SP2, SW9 to UP1, J14 to VIN1, J13 to VIN2, SW2 to X1, SW1 to Y1
Connections:
- J18 pad 1: /Pad2 -> SDA2
- J18 pad 2: /Pad1 -> SCL2
- J18 pad 3: VCC -> GND2
- TRACK_B2 pad 1: VCC -> /TB_in2
Routing:
- net VCC: track 5.22 -> 134.5 mm, vias 6 -> 7
- net GND2: track 43.9 -> 110.1 mm, vias 6 -> 5
- net GND: track 28.8 -> 94.6 mm, vias 2 -> 6
- net VCC2: track 49.5 -> 91.4 mm
- net 3.3v2: track 0.00 -> 14.1 mm
- net SCL2: track 54.9 -> 68.5 mm
- net 3.3V1: track 0.00 -> 12.9 mm, vias 0 -> 2
- net SCL: track 25.5 -> 32.0 mm
- net /Pad1: track 43.3 -> 37.1 mm, vias 2 -> 0
- net SDA2: track 68.8 -> 74.8 mm, vias 0 -> 2
- net SDA: track 27.7 -> 32.9 mm
- net /A32: track 34.0 -> 39.0 mm
- net /TB_in2: track 0.00 -> 4.27 mm
- net /L1: track 35.3 -> 31.3 mm
- net /PPVCC1: track 17.1 -> 21.0 mm
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Other:
- board size 130.9 x 105.1 mm -> 120 x 95.5 mm
