File: PCB/controller_Proto/contProto2/contProto.kicad_sch (KiCad schematic)
At the start: 78 parts, among them J1 JST_1mm_4, J10 JST_1mm_3, J11 JST_1mm_3, J12 Conn_01x03_Socket, J13 Conn_01x02_Socket, J14 Conn_01x02_Socket, J15 Conn_01x04, J16 Conn_01x04, J17 Conn_01x10_Pin, J18 JST_1mm_3, J19 Conn_01x08_Socket, J2 Conn_01x04, J22 JST_1mm_4, J23 Conn_01x03_Socket, J24 Conn_01x03_Socket, J25 Conn_01x03_Socket, J26 Conn_01x03_Socket, J27 Conn_01x03_Socket, J28 Conn_01x12_Socket, J29 Conn_01x12_Socket, J3 Conn_01x10_Pin, J30 Conn_01x12_Socket, J31 Conn_01x12_Socket, J32 Conn_01x03_Socket, J33 Conn_01x03_Socket, J36 Conn_01x05, J37 Conn_01x05, J4 JST_1mm_3, J5 Conn_01x02_Socket, J6 JST_1mm_3, J7 Conn_01x02_Socket, J9 Conn_01x04, SW1 SMD_12x12mm_h8.5mm, SW10 SMD_12x12mm_h8.5mm, SW11 SMD_12x12mm_h8.5mm, SW12 SMD_12x12mm_h8.5mm, SW13 SMD_12x12mm_h8.5mm, SW14 SMD_12x12mm_h8.5mm, SW15 SMD_12x12mm_h8.5mm, SW16 SMD_12x12mm_h8.5mm, SW17 SMD_12x12mm_h8.5mm, SW18 SMD_12x12mm_h8.5mm, SW19 SMD_12x12mm_h8.5mm, SW2 SMD_12x12mm_h8.5mm, SW20 SMD_12x12mm_h8.5mm, SW3 SMD_12x12mm_h8.5mm, SW4 SMD_12x12mm_h8.5mm, SW5 SMD_12x12mm_h8.5mm, SW6 SMD_12x12mm_h8.5mm, SW7 SMD_12x12mm_h8.5mm, SW8 SMD_12x12mm_h8.5mm, SW9 SMD_12x12mm_h8.5mm, U1 ProMicroC, U2 ProMicroC, U3 DRV5033FAxLPG, U4 DRV5033FAxLPG

Commit message: MAJOR PCB REDESIGN
shit here we go again
Connections:
- net Xout: now also J29.6 (Pin_6), U1.18 (A1); no longer J29.5 (Pin_5), U1.17 (A0)
- net Yout: now also J29.5 (Pin_5), U1.17 (A0); no longer J29.6 (Pin_6), U1.18 (A1)
Changed lines of the file:
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@@
-		)
-	)
-	(label "Yout"
-		(at 63.5 60.96 0)
-		(effects
-			(font
-				(size 1.27 1.27)
-			)
-			(justify left bottom)
 		)
 	)
@@
 		)
 	)
-	(label "Xout"
-		(at 55.88 22.86 270)
-		(effects
-			(font
-				(size 1.27 1.27)
-			)
-			(justify right bottom)
-		)
-	)
 	(label "U"
 		(at 177.8 31.75 180)
@@
 		)
 	)
+	(label "Yout"
+		(at 63.5 58.42 0)
+		(effects
+			(font
+				(size 1.27 1.27)
+			)
+			(justify left bottom)
+		)
+	)
 	(label "RST1"
 		(at 184.15 138.43 180)
@@
 		)
 	)
-	(label "Yout"
-		(at 58.42 22.86 270)
-		(effects
-			(font
-				(size 1.27 1.27)
-			)
-			(justify right bottom)
-		)
-	)
 	(label "PP22"
 		(at 212.09 59.69 180)
@@
 		)
 	)
+	(label "Xout"
+		(at 63.5 60.96 0)
+		(effects
+			(font
+				(size 1.27 1.27)
+			)
+			(justify left bottom)
+		)
+	)
 	(label "RST1"
 		(at 151.13 24.13 180)
@@
 		)
 	)
+	(label "Yout"
+		(at 55.88 22.86 270)
+		(effects
+			(font
+				(size 1.27 1.27)
+			)
+			(justify right bottom)
+		)
+	)
 	(label "U"
 		(at 59.69 160.02 270)
@@
 		)
 	)
-	(label "Xout"
-		(at 63.5 58.42 0)
-		(effects
-			(font
-				(size 1.27 1.27)
-			)
-			(justify left bottom)
-		)
-	)
 	(label "PPGND"
 		(at 203.2 138.43 270)
@@
 		(effects
 			(font
+				(size 1.27 1.27)
+			)
+			(justify right bottom)
+		)
+	)
+	(label "Xout"
+		(at 58.42 22.86 270)
+		(effects
+			(font

Commit message: final resesign and silk screen
Parts:
- removed TP1, TP4: TestPoint_2Pole, TestPoint:TestPoint_Bridge_Pitch2.0mm_Drill0.7mm, symbol Connector:TestPoint_2Pole
- added J20, J8: JST_1mm_4, Connector_JST:JST_GH_BM04B-GHS-TBT_1x04-1MP_P1.25mm_Vertical, symbol PCM_SparkFun-Connector:Conn_01x04_JST_P1.0mm_Horizontal_SMD
- J1, J22: footprint PCM_SparkFun-Connector:JST_1x04_P1.0mm_Horizontal_SMD -> Connector_JST:JST_GH_BM04B-GHS-TBT_1x04-1MP_P1.25mm_Vertical
Connections:
- net Btn_-: now also R22.1, J8.4
- net Btn_SP3: now also R9.1, J8.3
- net GND2: now also J31.2 (Pin_2), J20.2; no longer R22.2, R9.2
- net R: now also SW11.1
- net SP2: now also J29.2 (Pin_2), U1.14 (D16); no longer J29.1 (Pin_1), U1.13 (D10/A10)
- net SP3: now also J20.3; no longer R9.1
- net VCC2: now also J20.1; no longer SW12.2, SW14.2
- net minus: now also J20.4; no longer R22.1
- net plus: now also J29.1 (Pin_1), U1.13 (D10/A10); no longer J29.2 (Pin_2), U1.14 (D16)
- new net SL_GND: J8.2, R22.2, R9.2
- new net SL_VCC: J8.1, SW12.2, SW14.2

Commit message: final pcb
Parts:
- removed J1, J20, J22, J8: JST_1mm_4, Connector_JST:JST_GH_BM04B-GHS-TBT_1x04-1MP_P1.25mm_Vertical, symbol PCM_SparkFun-Connector:Conn_01x04_JST_P1.0mm_Horizontal_SMD
- removed J15, J16, J2: Conn_01x04, Connector_JST:JST_GH_BM04B-GHS-TBT_1x04-1MP_P1.25mm_Vertical, symbol PCM_SparkFun-Connector:Conn_01x04_JST_P2.0mm_Horizontal_SMD
- removed J36: Conn_01x05, Connector_JST:JST_GH_BM05B-GHS-TBT_1x05-1MP_P1.25mm_Vertical, symbol PCM_SparkFun-Connector:Conn_01x05_JST_P1.0mm_Horizontal_SMD
- removed J6: JST_1mm_3, Connector_JST:JST_GH_BM03B-GHS-TBT_1x03-1MP_P1.25mm_Vertical, symbol PCM_SparkFun-Connector:Conn_01x03_JST_P1.0mm_Horizontal_SMD
- added JP1, JP2: ~, PCM_SparkFun-Jumper:Jumper_3_NO, symbol PCM_SparkFun-Jumper:SolderJumper_3_Open
- added L_SHOUL1, PAD3, PAD4, PAD_B1, PAD_B2, R_SHOUL1, R_SHOULD1, SP_L1, SP_LB1: Conn_01x04, Connector_FFC-FPC:Amphenol_F32Q-1A7x1-11004_1x04-1MP_P0.5mm_Horizontal, symbol PCM_SparkFun-Connector:Conn_01x04_JST_P2.0mm_Horizontal_SMD
- added R12, R23, R24, R25, R26, R27: 1k, PCM_SparkFun-Resistor:R_0805_2012Metric, symbol PCM_SparkFun-Resistor:1k_0402
- added TRACK_B1: Conn_01x05, Connector_PinHeader_2.54mm:PinHeader_1x05_P2.54mm_Vertical, symbol PCM_SparkFun-Connector:Conn_01x05_JST_P1.0mm_Horizontal_SMD
- J11: footprint Connector_JST:JST_GH_BM03B-GHS-TBT_1x03-1MP_P1.25mm_Vertical -> Connector_PinHeader_2.54mm:PinHeader_1x03_P2.54mm_Vertical
- J9: footprint Connector_JST:JST_GH_BM04B-GHS-TBT_1x04-1MP_P1.25mm_Vertical -> Connector_FFC-FPC:Amphenol_F32Q-1A7x1-11004_1x04-1MP_P0.5mm_Horizontal
- R1, R10, R13, R14, R15, R16, R17, R18, R19, R2, R20, R21, R22, R3, R4, R5, R6, R7, R8, R9: footprint PCM_SparkFun-Resistor:R_0402_1005Metric -> PCM_SparkFun-Resistor:R_0805_2012Metric
- RUMBLE1: renamed from J10; footprint Connector_JST:JST_GH_BM03B-GHS-TBT_1x03-1MP_P1.25mm_Vertical -> Connector_PinHeader_2.54mm:PinHeader_1x03_P2.54mm_Vertical
- TRACK_B2: renamed from J37; value Conn_01x05 -> TRACK_B; footprint Connector_JST:JST_GH_BM05B-GHS-TBT_1x05-1MP_P1.25mm_Vertical -> Connector_PinHeader_2.54mm:PinHeader_1x05_P2.54mm_Vertical
- renumbered SW4 to A1, SW3 to B1, J5 to CAP1, J7 to CAP2, SW10 to DWN1, J4 to I2C1, J3 to JOY_R1, SW8 to L1, SW16 to LB1, U3 to LT1, SW12 to MINUS1, J19 to MPU1, SW13 to PAD1, SW6 to PAD2, SW5 to PLUS1, SW11 to R11, SW15 to RB1, SW17 to RST1, SW18 to RST2, U4 to RT1, SW7 to SP1, SW14 to SP2, SW9 to UP1, J14 to VIN1, J13 to VIN2, SW2 to X1, SW1 to Y1
Connections:
- net 5V: now also JP2.1 (A), PAD3.2, R12.1, R_SHOULD1.1; no longer J18.3, TRACK_B2.1
- net Btn_-: now also SP_LB1.3
- net Btn_SP3: now also SP_LB1.4
- net GND: now also PAD3.1, R26.2, R_SHOULD1.2
- net GND2: now also J18.3, PAD4.1, R27.2, SP_L1.1, TRACK_B1.5
- net GND_LSP: now also L_SHOUL1.2
- net GND_RSP: now also R_SHOUL1.2
- net L1P: now also L_SHOUL1.3
- net L2P: now also L_SHOUL1.4
- net PP1: now also PAD_B1.3
- net PP2: now also PAD_B1.4
- net PP3: now also PAD_B2.3
- net PP4: now also PAD_B2.4
- net PPGND: now also PAD_B1.1
- net PPGND2: now also PAD_B2.1
- net PPVCC1: now also PAD_B1.2
- net PPVCC2: now also PAD_B2.2
- net Pad1: now also PAD3.3; no longer J18.2
- net Pad2: now also PAD3.4; no longer J18.1
- net Pad3: now also PAD4.3
- net Pad4: now also PAD4.4
- net R1: now also R_SHOULD1.3
- net R1P: now also R_SHOUL1.3
- net R2: now also R_SHOULD1.4
- net R2P: now also R_SHOUL1.4
- net SCL2: now also J18.2, TRACK_B1.2
- net SDA2: now also J18.1, TRACK_B1.3
- net SL_GND: now also SP_LB1.1
- net SL_VCC: now also SP_LB1.2
- net SP3: now also SP_L1.4
- net VCC2: now also JP1.1 (A), PAD4.2, R24.1, SP_L1.2
- net VCC_LSP: now also L_SHOUL1.1
- net VCC_RSP: now also R_SHOUL1.1
- net minus: now also SP_L1.3
- new net: R25.2, R27.1
- new net: R23.2, R26.1
- new net 3.3V1: JP2.3 (C), R12.2, R23.1
- new net 3.3v2: JP1.3 (C), R24.2, R25.1
- new net TB_in: JP1.2 (B), TRACK_B1.1
- new net TB_in2: JP2.2 (B), TRACK_B2.1
